File: Probe instrumentation/PAINTREv3/PAINTREv3.kicad_sch (KiCad schematic)
At the start: 97 parts

Commit message: V4
Parts:
- C1, C11, C12, C14, C17, C18, C19, C2, C20, C22, C23, C26, C27, C28, C29, C30, C4, C9: value (none) -> .1u; footprint (none) -> Capacitor_SMD:C_0603_1608Metric_fabdesignatorsmall
- C10, C13, C15, C16, C21, C24, C25, C3, C8: value (none) -> 1u; footprint (none) -> Capacitor_SMD:C_0603_1608Metric_fabdesignatorsmall
- C5: value (none) -> 10n; footprint (none) -> Capacitor_SMD:C_0603_1608Metric_fabdesignatorsmall
- C6, C7: value (none) -> 10u; footprint (none) -> New folder:C_1206_HandSoldering_silkscreenlabel
- D7: value (none) -> AQ12; footprint (none) -> TO_SOT_Packages_SMD:SOT-23_handsoldering
- F1: value (none) -> Polyfuse; footprint (none) -> Fuse:Fuse_0603_1608Metric
- H1, H2: value (none) -> MountingHole; footprint (none) -> MountingHole:MountingHole_3.2mm_M3
- J1: value (none) -> ethernet; footprint (none) -> Connector_PinSocket_2.00mm:PinSocket_1x08_P2.00mm_Vertical
- J2: value (none) -> SPI; footprint (none) -> Connectors_JST:JST_SH_SM04B-SRSS-TB_04x1.00mm_Angled
- J3: value (none) -> TC; footprint (none) -> Connector_PinHeader_2.54mm:ScrewTerminal_1x12_P2.54mm_Vertical
- J5: value (none) -> debug; footprint (none) -> Connectors_JST:JST_SH_SM04B-SRSS-TB_04x1.00mm_Angled
- J7: value (none) -> BN080; footprint (none) -> Connectors_JST:JST_SH_SM04B-SRSS-TB_04x1.00mm_Angled
- L5, L6: value (none) -> Ferrite_Bead_Small; footprint (none) -> New folder:ferrite_bead_handsolder-1206
- R1, R12, R16, R2, R20, R22, R25, R27, R28, R29, R3, R30, R31, R4, R40: value (none) -> 1M; footprint (none) -> Resistor_SMD:R_0603_1608Metric_fabdesignatorsmall
- R10, R11, R17, R18, R19, R21, R26, R36, R37, R38, R39, R9, Rterm1, Rterm2: value (none) -> 50; footprint (none) -> Resistor_SMD:R_0603_1608Metric_fabdesignatorsmall
- R13, R15, R23, R24, R32, R33, R34, R35, R5, R6, R7, R8, Ri2cSCL1, Ri2cSCL2, Ri2cSDA1, Ri2cSDA2: value (none) -> 500; footprint (none) -> Resistor_SMD:R_0603_1608Metric_fabdesignatorsmall
- R14: value (none) -> 4.7k; footprint (none) -> Resistor_SMD:R_0603_1608Metric_fabdesignatorsmall
- TP2: value (none) -> pc0; footprint (none) -> TestPoint:TestPoint_Pad_2.0x2.0mm
- TP3: value (none) -> pc1; footprint (none) -> TestPoint:TestPoint_Pad_2.0x2.0mm
- TP4: value (none) -> pc2; footprint (none) -> TestPoint:TestPoint_Pad_2.0x2.0mm
- U1: value (none) -> LP2985-3.3; footprint (none) -> TO_SOT_Packages_SMD:SOT-23-5_HandSoldering
- U2: value (none) -> THVD1428DR; footprint (none) -> Package_SO:SOIC-8_3.9x4.9mm_P1.27mm
- U3, U4, U7: value (none) -> ADS1118IDGS; footprint (none) -> Package_SO:TSSOP-10_3x3mm_P0.5mm
- U5: value (none) -> ATmega328P-AU; footprint (none) -> Housings_QFP:TQFP-32_7x7mm_Pitch0.8mm
- Y1: value (none) -> 8MHz Resonator; footprint (none) -> New folder:Resonator_SMD_muRata_CSTNE
Other:
- note added: "<.2mA each"
