File: Probe instrumentation/PAINTREv4/_autosave-PAINTREv4.kicad_pcb (KiCad board)
At the start: 4 copper layers, 20 x 94.7 mm, 113 parts, among them J1 ethernet, J3 TC, J7 BN080, U1 LP2985-5.0, U3 ADS1118IDGS, U4 ADS1118IDGS, U5 ADS1118IDGS, U7 ADS1118IDGS

Commit message: update pre-arduino
Parts:
- added D7: AQ12, Library:SOT-23_handsoldering, F.Cu at (130.2, 70.1)
- added L1: ~, Library:ferrite_bead_1206, F.Cu at (134.7, 83.6)
- added REF**: Arduino_Nano, Module:Arduino_Nano, F.Cu at (157.6, 49.3)
- moved L5 2.10 mm to (126.9, 70.7)
Routing:
- net Net-(C3-Pad1): track 6.79 -> 34.5 mm, vias 0 -> 3
- net Net-(D7-Pad1): track 6.15 -> 10.8 mm
- net UART_TX: track 16.5 -> 17.7 mm, vias 0 -> 2
- net UART_RX: track 14.7 -> 15.7 mm, vias 0 -> 2
- net GND: track 98.7 -> 99.5 mm, vias 51 -> 50
- net Net-(C16-Pad1): track 8.14 -> 8.70 mm
