File: Probe instrumentation/PAINTREv4/PAINTREv4.kicad_pcb (KiCad board)
At the start: 4 copper layers, 20 x 94.7 mm, 113 parts, among them J1 ethernet, J3 TC, J7 BN080, U1 LP2985-5.0, U3 ADS1118IDGS, U4 ADS1118IDGS, U5 ADS1118IDGS, U7 ADS1118IDGS

Commit message: arduino version
Parts:
- removed C16: 1u, Library:C_0603_1608Metric_fabdesignatorsmall
- removed C3, C4, C5: ~, Library:C_0603_1608Metric_fabdesignatorsmall
- removed C35: 10n, Library:C_0603_1608Metric_fabdesignatorsmall
- removed C6: 10u, Library:C_1206_HandSoldering_silkscreenlabel
- removed J5: ~, Library:Tag-Connect_TC2030-IDC-NL_2x03_P1.27mm_Vertical
- removed U1: LP2985-5.0, Package_TO_SOT_SMD:SOT-23-5
- removed U2: ~, Package_QFP:TQFP-48_7x7mm_P0.5mm
- added A1: Arduino_Nano_Every, Module:Arduino_Nano, F.Cu at (127.0, 55.0)
- added D7: AQ12, Library:SOT-23_handsoldering, F.Cu at (129.9, 38.9)
- moved C7 37.5 mm to (134.0, 46.0)
- moved L5 31.3 mm to (126.6, 39.5)
- moved R56 31.2 mm to (139.2, 38.8)
- moved C36 31.2 mm to (136.5, 39.5)
- moved J1 31.2 mm to (128.7, 34.0)
- moved R54 31.2 mm to (139.9, 49.0)
- moved R55 31.2 mm to (141.1, 38.8)
- moved R57 31.2 mm to (140.0, 36.3)
- moved U6 31.2 mm to (140.1, 44.3)
- moved R53 31.2 mm to (136.5, 44.3)
- moved F1 14.0 mm to (135.4, 102.6)
- moved J7 12.9 mm to (140.5, 101.4), turned to 90 degrees
- moved Ri2cSDA2 10.9 mm to (132.3, 100.8)
- moved Ri2cSDA1 10.9 mm to (135.4, 100.8)
- moved Ri2cSCL1 8.37 mm to (135.4, 99.2)
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Connections:
- L5 pad 1: Net-(C16-Pad1) -> Vin
Routing:
- net Vin: track 0.00 -> 24.7 mm
- net GND: track 98.7 -> 78.9 mm, vias 51 -> 43
- net sda: track 23.7 -> 4.32 mm, vias 2 -> 0
- net scl: track 18.9 -> 4.30 mm
- net cipo: track 77.5 -> 65.4 mm, vias 7 -> 4
- net +5V: track 72.6 -> 60.5 mm, vias 23 -> 21
- net RXD: track 11.6 -> 0.00 mm, vias 2 -> 0
- net copi: track 75.6 -> 64.5 mm, vias 7 -> 4
- net UART_RX: track 14.7 -> 3.64 mm, vias 0 -> 1
- net Net-(F1-Pad2): track 12.6 -> 2.06 mm, vias 2 -> 1
- net UART_TX: track 16.5 -> 6.01 mm, vias 0 -> 1
- net cs_2: track 57.9 -> 67.6 mm, vias 4 -> 3
- net RS485_EN: track 14.9 -> 5.49 mm, vias 2 -> 1
- net cs_3: track 47.3 -> 56.4 mm, vias 2 -> 3
- net TXD: track 9.04 -> 0.00 mm
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Other:
- board size 20 x 94.7 mm -> 20 x 125.9 mm

Commit message: V4 PCB redesign (max ICs)
Parts:
- removed C10, C12, C21, C24, C33: 1u, Library:C_0603_1608Metric_fabdesignatorsmall
- removed C11, C13, C14, C15, C23, C30, C31, C32: .1u, Library:C_0603_1608Metric_fabdesignatorsmall
- removed R10, R11, R19, R21, R26, R36, R37, R38, R39, R48, R49, R50, R51, R9: 50, Library:R_0603_1608Metric_fabdesignatorsmall
- removed R12, R22, R25, R27, R28, R29, R30, R31, R40, R41, R42, R43, R52: 1M, Library:R_0603_1608Metric_fabdesignatorsmall
- removed R32, R33, R34, R35, R44, R45, R46, R47, R7, R8: 500, Library:R_0603_1608Metric_fabdesignatorsmall
- removed U7: ADS1118IDGS, Package_SO:TSSOP-10_3x3mm_P0.5mm
- added C16: .1u, Library:C_0603_1608Metric_fabdesignatorsmall, F.Cu at (133.2, 132.7)
- added C3: .1u, Library:C_0603_1608Metric_fabdesignatorsmall, F.Cu at (135.9, 125.7)
- added C4: .1u, Library:C_0603_1608Metric_fabdesignatorsmall, F.Cu at (135.9, 129.0)
- added C5: .1u, Library:C_0603_1608Metric_fabdesignatorsmall, F.Cu at (135.9, 117.4)
- added C6: .1u, Library:C_0603_1608Metric_fabdesignatorsmall, F.Cu at (135.9, 120.7)
- added J2: TC1, Connector_PinSocket_2.54mm:PinSocket_1x02_P2.54mm_Vertical, F.Cu at (142.0, 145.8)
- added J4: TC3, Connector_PinSocket_2.54mm:PinSocket_1x02_P2.54mm_Vertical, F.Cu at (142.0, 126.2)
- added J5: TC4, Connector_PinSocket_2.54mm:PinSocket_1x02_P2.54mm_Vertical, F.Cu at (142.0, 117.7)
- added J6: TC5, Connector_PinSocket_2.54mm:PinSocket_1x02_P2.54mm_Vertical, F.Cu at (142.0, 109.8)
- added U1: MAX31855KASA, Package_SO:SOIC-8_3.9x4.9mm_P1.27mm, F.Cu at (130.9, 145.0)
- added U2: MAX31855KASA, Package_SO:SOIC-8_3.9x4.9mm_P1.27mm, F.Cu at (130.9, 136.4)
- C25: value 1u -> .01u
- C26, C27, C28, C29: value .1u -> .01u
- C8, C9: value 1u -> .1u
- J3: value TC -> TC2; footprint Connector_PinHeader_2.54mm:PinHeader_1x16_P2.54mm_Vertical -> Connector_PinSocket_2.54mm:PinSocket_1x02_P2.54mm_Vertical
- R1, R2, R3, R4: value 1M -> 500
- R17, R18: value 50 -> 1M
- U3, U4, U5: value ADS1118IDGS -> MAX31855KASA; footprint Package_SO:TSSOP-10_3x3mm_P0.5mm -> Package_SO:SOIC-8_3.9x4.9mm_P1.27mm
- U6: footprint Package_SO:SOIC-8_3.9x4.9mm_P1.27mm -> Library:SOT-5X3-8
- moved R18 40.9 mm to (129.8, 107.8), turned to 0 degrees
- moved R17 38.3 mm to (129.8, 116.3), turned to 0 degrees
- moved C8 33.0 mm to (135.9, 109.4), turned to -90 degrees
- moved R5 32.1 mm to (138.4, 108.7)
- moved C19 29.5 mm to (133.1, 107.8)
- moved R6 28.9 mm to (138.4, 113.5)
- moved R16 27.5 mm to (129.9, 124.0), turned to 0 degrees
- moved C25 22.0 mm to (138.5, 144.5), turned to 180 degrees
- moved R14 20.6 mm to (129.8, 132.7)
- moved C17 20.1 mm to (133.2, 124.0)
- moved C18 17.9 mm to (133.2, 116.3)
- moved J3 17.6 mm to (142.0, 134.6), turned to 0 degrees
- moved R3 16.0 mm to (138.4, 116.6), turned to 180 degrees
- moved R4 15.9 mm to (138.4, 121.5)
- moved U3 14.4 mm to (130.9, 127.7), turned to 180 degrees
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Connections:
- A1 pad 10: cs_1 -> cs_2
- A1 pad 11: cs_2 -> cs_3
- A1 pad 12: cs_3 -> cs_4
- A1 pad 13: cs_4 -> cs_5
- A1 pad 9: unconnected-(A1-Pad9) -> cs_1
- C17 pad 1: Net-(C17-Pad1) -> +5V
- C18 pad 1: GND -> +5V
- C18 pad 2: Net-(C10-Pad1) -> GND
- C19 pad 1: Net-(C10-Pad2) -> +5V
- C22 pad 1: Net-(C21-Pad2) -> Net-(C22-Pad1)
- C25 pad 1: Net-(C25-Pad1) -> Net-(C20-Pad2)
- C25 pad 2: Net-(C25-Pad2) -> Net-(C22-Pad1)
- C26 pad 1: GND -> Net-(C3-Pad2)
- C26 pad 2: Net-(C24-Pad1) -> Net-(C4-Pad1)
- C27 pad 1: Net-(C24-Pad2) -> Net-(C2-Pad2)
- C27 pad 2: GND -> Net-(C34-Pad1)
- C28 pad 1: GND -> Net-(C5-Pad2)
- C28 pad 2: Net-(C25-Pad1) -> Net-(C6-Pad1)
- C29 pad 1: Net-(C25-Pad2) -> Net-(C8-Pad2)
- C29 pad 2: GND -> Net-(C9-Pad1)
- C34 pad 1: Net-(C33-Pad2) -> Net-(C34-Pad1)
- C8 pad 1: Net-(C11-Pad2) -> GND
- C8 pad 2: Net-(C17-Pad1) -> Net-(C8-Pad2)
- C9 pad 1: Net-(C13-Pad2) -> Net-(C9-Pad1)
- C9 pad 2: Net-(C14-Pad1) -> GND
- J3 pad 1: tc1- -> tc2+
- J3 pad 2: tc1+ -> tc2-
- R1 pad 1: +5V -> tc3+
- R1 pad 2: tc3+ -> Net-(C3-Pad2)
- R14 pad 1: +5V -> cs_2
- R14 pad 2: tc7+ -> +5V
- R15 pad 2: Net-(C33-Pad2) -> Net-(C34-Pad1)
- R16 pad 1: tc2- -> cs_3
- R16 pad 2: GND -> +5V
- R17 pad 1: Net-(R17-Pad1) -> cs_4
- R17 pad 2: sck -> +5V
- R18 pad 1: Net-(R18-Pad1) -> cs_5
- R18 pad 2: copi -> +5V
- R2 pad 2: GND -> Net-(C4-Pad1)
- R24 pad 2: Net-(C21-Pad2) -> Net-(C22-Pad1)
- R3 pad 1: +5V -> tc4+
- R3 pad 2: tc4+ -> Net-(C5-Pad2)
- R4 pad 2: GND -> Net-(C6-Pad1)
- R5 pad 1: tc3+ -> tc5+
- R5 pad 2: Net-(C11-Pad2) -> Net-(C8-Pad2)
- R6 pad 1: tc3- -> tc5-
- R6 pad 2: Net-(C17-Pad1) -> Net-(C9-Pad1)
- U3 pad 1: Net-(R9-Pad1) -> GND
- U3 pad 2: Net-(R26-Pad1) -> Net-(C4-Pad1)
- U3 pad 3: GND -> Net-(C3-Pad2)
- U3 pad 4: Net-(C11-Pad2) -> +5V
- U3 pad 5: Net-(C17-Pad1) -> sck
- U3 pad 6: Net-(C10-Pad1) -> cs_3
- U3 pad 7: Net-(C10-Pad2) -> cipo
- U3 pad 8: +5V -> (no net)
- U4 pad 1: Net-(R36-Pad1) -> GND
- U4 pad 2: Net-(R39-Pad1) -> Net-(C6-Pad1)
- U4 pad 3: GND -> Net-(C5-Pad2)
- U4 pad 4: Net-(C24-Pad1) -> +5V
- U4 pad 5: Net-(C24-Pad2) -> sck
- U4 pad 6: Net-(C25-Pad1) -> cs_4
- U4 pad 7: Net-(C25-Pad2) -> cipo
- U4 pad 8: +5V -> (no net)
- U5 pad 1: Net-(R48-Pad1) -> GND
- U5 pad 2: Net-(R51-Pad1) -> Net-(C9-Pad1)
- U5 pad 3: GND -> Net-(C8-Pad2)
- U5 pad 4: Net-(C13-Pad2) -> +5V
- U5 pad 5: Net-(C14-Pad1) -> sck
- U5 pad 6: Net-(C12-Pad1) -> cs_5
- U5 pad 7: Net-(C12-Pad2) -> cipo
- U5 pad 8: +5V -> (no net)
Routing:
- net copi: track 64.5 -> 0.00 mm, vias 4 -> 0
- net GND: track 78.9 -> 42.0 mm, vias 43 -> 19
- net cs_5: track 0.00 -> 33.5 mm, vias 0 -> 2
- net +5V: track 60.5 -> 37.3 mm, vias 21 -> 7
- net Net-(C12-Pad2): track 11.1 -> 0.00 mm
- net Net-(C25-Pad2): track 11.1 -> 0.00 mm
- net Net-(C12-Pad1): track 9.85 -> 0.00 mm
- net Net-(C25-Pad1): track 9.82 -> 0.00 mm
- net Net-(C10-Pad2): track 9.63 -> 0.00 mm
- net tc8+: track 9.00 -> 0.00 mm
- net Net-(C10-Pad1): track 8.74 -> 0.00 mm
- net tc8-: track 8.56 -> 0.00 mm
- net Net-(C3-Pad2): track 0.00 -> 8.14 mm
- net Net-(C5-Pad2): track 0.00 -> 8.14 mm
- net Net-(C13-Pad2): track 8.04 -> 0.00 mm
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
Commit message: v4 pcb updates
Parts:
- moved H1 66.2 mm to (126.4, 46.2)
- moved C36 5.66 mm to (138.0, 45.0), turned to 90 degrees
- moved H3 3.58 mm to (142.0, 151.4)
- moved R53 0.82 mm to (136.0, 45.0)
- moved C19 0.66 mm to (133.1, 107.2)
- moved C29 0.66 mm to (138.4, 110.3)
- moved C8 0.66 mm to (135.9, 108.8)
- moved C9 0.66 mm to (135.9, 112.1)
- moved J6 0.66 mm to (142.0, 109.1)
- moved R18 0.66 mm to (129.8, 107.2)
- moved R5 0.66 mm to (138.4, 108.0)
- moved R6 0.66 mm to (138.4, 112.9)
- moved U5 0.66 mm to (130.9, 110.8)
- moved C18 0.53 mm to (133.2, 115.8)
- moved R17 0.53 mm to (129.8, 115.8)
Routing:
- net GND: track 42.0 -> 82.8 mm, vias 19 -> 31
- net scl: track 0.95 -> 33.9 mm, vias 0 -> 1
- net sda: track 1.09 -> 32.5 mm, vias 0 -> 1
- net RS485_EN: track 5.49 -> 36.5 mm
- net UART_RX: track 3.64 -> 22.6 mm
- net UART_TX: track 6.01 -> 22.0 mm
- net +5V: track 37.3 -> 52.7 mm, vias 7 -> 14
- net Net-(C9-Pad1): track 5.35 -> 7.77 mm
- net Net-(R56-Pad2): track 2.33 -> 4.34 mm
- net Net-(C8-Pad2): track 5.60 -> 7.52 mm
- net Net-(R55-Pad2): track 2.43 -> 4.23 mm
- net Net-(F1-Pad2): track 1.40 -> 2.70 mm, vias 1 -> 0
- net sck: track 73.7 -> 74.2 mm
Other:
- board size 20 x 125.9 mm -> 20 x 121.5 mm
- board text added: "1"
- board text added: "2"
- board text added: "3"
- board text added: "4"
- board text added: "5"
- board text added: "A"
- board text added: "B"
- board text added: "THVD1400"
- board text removed: "L5 L6"

Commit message: pv4
Parts:
- C36: value ~ -> .1u
- H2: value MountingHole -> logo; footprint Library:MountingHole_3.2mm_M3 -> Library:paintre v4 logo
- R57: footprint Library:R_0603_1608Metric_fabdesignatorsmall -> Resistor_SMD:R_1210_3225Metric_Pad1.30x2.65mm_HandSolder
- moved H2 48.2 mm to (135.0, 73.0)
- moved R56 1.74 mm to (139.2, 40.5)
- moved R55 1.74 mm to (141.1, 40.5)
- moved H1 1.70 mm to (127.9, 47.0)
- moved R57 0.84 mm to (139.8, 37.1)
Routing:
- net RS485_A-: track 6.40 -> 8.49 mm
- net RS485_B+: track 6.42 -> 8.24 mm
- net Net-(R56-Pad2): track 4.34 -> 2.60 mm
- net Net-(R55-Pad2): track 4.23 -> 2.49 mm
Other:
- board text added: "PAINTRE v4"
- board text added: "Rt"
- board text added: "clan@geus.dk"
- board text removed: "BNO080"
- board text removed: "J2"
- board text removed: "J5"
