File: Probe instrumentation/PAINTREv4/PAINTREv4.kicad_sch (KiCad schematic)
At the start: 117 parts, among them J1 ethernet, J3 TC, J7 BN080, U1 LP2985-5.0, U3 ADS1118IDGS, U4 ADS1118IDGS, U5 ADS1118IDGS, U7 ADS1118IDGS

Commit message: update pre-arduino
Parts:
- removed JPWR1, RS4851: ~, symbol Connector:Conn_01x02_Female
- D7: footprint TO_SOT_Packages_SMD:SOT-23_handsoldering -> Library:SOT-23_handsoldering
- L1: footprint (none) -> Library:ferrite_bead_1206
- L5: footprint New folder:ferrite_bead_handsolder-1206 -> Library:ferrite_bead_1206
Connections:
- net RS485_EN: now also U2.37 (PF3); no longer U2.48 (PA4)
Changed lines of the file:
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@@
     )
   )
-  (global_label "Vin" (shape input) (at 325.12 242.57 90) (fields_autoplaced)
-    (effects (font (size 1.27 1.27)) (justify left))
-    (property "Intersheet References" "${INTERSHEET_REFS}" (id 0) (at 227.33 34.29 0)
-      (effects (font (size 1.27 1.27)) hide)
-    )
-  )
   (global_label "copi" (shape input) (at 172.72 125.73 180) (fields_autoplaced)
     (effects (font (size 1.27 1.27)) (justify right))
@@
     )
   )
-  (global_label "RS485_A-" (shape input) (at 342.9 245.11 0) (fields_autoplaced)
-    (effects (font (size 1.27 1.27)) (justify left))
-    (property "Intersheet References" "${INTERSHEET_REFS}" (id 0) (at 227.33 34.29 0)
-      (effects (font (size 1.27 1.27)) hide)
-    )
-  )
   (global_label "UART_TX" (shape input) (at 199.39 63.5 180) (fields_autoplaced)
     (effects (font (size 1.27 1.27)) (justify right))
@@
     )
   )
-  (global_label "RS485_B+" (shape input) (at 342.9 242.57 0) (fields_autoplaced)
-    (effects (font (size 1.27 1.27)) (justify left))
-    (property "Intersheet References" "${INTERSHEET_REFS}" (id 0) (at 227.33 34.29 0)
-      (effects (font (size 1.27 1.27)) hide)
-    )
-  )
   (global_label "RS485_EN" (shape input) (at 219.71 58.42 180) (fields_autoplaced)
     (effects (font (size 1.27 1.27)) (justify right))
@@
     )
   )
-  (global_label "RS485_EN" (shape input) (at 203.2 110.49 0) (fields_autoplaced)
-    (effects (font (size 1.27 1.27)) (justify left))
-    (property "Intersheet References" "${INTERSHEET_REFS}" (id 0) (at 50.8 2.54 0)
+  (global_label "RS485_EN" (shape input) (at 172.72 113.03 180) (fields_autoplaced)
+    (effects (font (size 1.27 1.27)) (justify right))
+    (property "Intersheet References" "${INTERSHEET_REFS}" (id 0) (at 325.12 220.98 0)
       (effects (font (size 1.27 1.27)) hide)
     )
@@
       (effects (font (size 1.27 1.27)) (justify left))
     )
-    (property "Footprint" "TO_SOT_Packages_SMD:SOT-23_handsoldering" (id 2) (at 43.18 27.94 0)
+    (property "Footprint" "Library:SOT-23_handsoldering" (id 2) (at 43.18 27.94 0)
       (effects (font (size 1.27 1.27)) hide)
     )
@@
       (effects (font (size 1.27 1.27)) hide)
     )
-    (property "Footprint" "New folder:ferrite_bead_handsolder-1206" (id 2) (at 54.61 23.622 90)
+    (property "Footprint" "Library:ferrite_bead_1206" (id 2) (at 54.61 23.622 90)
       (effects (font (size 1.27 1.27)) hide)
     )
@@
     (property "Reference" "L1" (id 0) (at 196.85 96.266 90))
     (property "Value" "~" (id 1) (at 196.85 93.9546 90))
-    (property "Footprint" "" (id 2) (at 196.85 91.44 0)
+    (property "Footprint" "Library:ferrite_bead_1206" (id 2) (at 196.85 91.44 0)
       (effects (font (size 1.27 1.27)) hide)
     )
@@
     )
   )
-  (symbol (lib_id "Connector:Conn_01x02_Female") (at 337.82 245.11 180) (unit 1)
-    (in_bom yes) (on_board yes)
-    (property "Reference" "RS4851" (id 0) (at 334.01 243.84 0))
-    (property "Value" "~" (id 1) (at 340.5632 239.1664 0)
-      (effects (font (size 1.27 1.27)) hide)
-    )
-    (property "Footprint" "" (id 2) (at 337.82 245.11 0)
-      (effects (font (size 1.27 1.27)) hide)
-    )
-    (property "Datasheet" "~" (id 3) (at 337.82 245.11 0)
-      (effects (font (size 1.27 1.27)) hide)
-    )
-    (property "JLC part number" "---" (id 4) (at 337.82 245.11 0)
-      (effects (font (size 1.27 1.27)) hide)
-    )
-    (pin "1")
-    (pin "2")
-  )
-  (symbol (lib_id "Connector:Conn_01x02_Female") (at 320.04 245.11 180) (unit 1)
-    (in_bom yes) (on_board yes)
-    (property "Reference" "JPWR1" (id 0) (at 316.23 243.84 0))
-    (property "Value" "~" (id 1) (at 322.7832 239.1664 0)
-      (effects (font (size 1.27 1.27)) hide)
-    )
-    (property "Footprint" "" (id 2) (at 320.04 245.11 0)
-      (effects (font (size 1.27 1.27)) hide)
-    )
-    (property "Datasheet" "~" (id 3) (at 320.04 245.11 0)
-      (effects (font (size 1.27 1.27)) hide)
-    )
-    (property "JLC part number" "---" (id 4) (at 320.04 245.11 0)
-      (effects (font (size 1.27 1.27)) hide)
-    )
-    (pin "1")
-    (pin "2")
-  )
-  (symbol (lib_id "power:GND") (at 325.12 245.11 0) (unit 1)
-    (in_bom yes) (on_board yes)
-    (property "Reference" "#PWR0168" (id 0) (at 325.12 251.46 0)
-      (effects (font (size 1.27 1.27)) hide)
-    )
-    (property "Value" "~" (id 1) (at 325.247 249.5042 0))
-    (property "Footprint" "" (id 2) (at 325.12 245.11 0)
-      (effects (font (size 1.27 1.27)) hide)
-    )
-    (property "Datasheet" "" (id 3) (at 325.12 245.11 0)
-      (effects (font (size 1.27 1.27)) hide)
-    )
-    (pin "1")
-  )
   (symbol (lib_id "Device:R") (at 257.81 30.48 0) (unit 1)
     (in_bom yes) (on_board yes)
@@
       (reference "#PWR0167") (unit 1) (value "+5V") (footprint "")
     )
-    (path "/00000000-0000-0000-0000-00006180a484"
-      (reference "#PWR0168") (unit 1) (value "~") (footprint "")
-    )
     (path "/00000000-0000-0000-0000-00006190a937"
       (reference "#PWR0169") (unit 1) (value "~") (footprint "")
@@
     )
     (path "/00000000-0000-0000-0000-00005dc455cc"
-      (reference "D7") (unit 1) (value "AQ12") (footprint "TO_SOT_Packages_SMD:SOT-23_handsoldering")
+      (reference "D7") (unit 1) (value "AQ12") (footprint "Library:SOT-23_handsoldering")
     )
     (path "/00000000-0000-0000-0000-000060094555"
@@
       (reference "J7") (unit 1) (value "BN080") (footprint "Library:JST_SH_SM04B-SRSS-TB_04x1.00mm_Angled")
     )
-    (path "/00000000-0000-0000-0000-000061808b52"
-      (reference "JPWR1") (unit 1) (value "~") (footprint "")
-    )
     (path "/00000000-0000-0000-0000-0000615f07b8"
-      (reference "L1") (unit 1) (value "~") (footprint "")
+      (reference "L1") (unit 1) (value "~") (footprint "Library:ferrite_bead_1206")
     )
     (path "/00000000-0000-0000-0000-00005de07c7e"
-      (reference "L5") (unit 1) (value "Ferrite_Bead_Small") (footprint "New folder:ferrite_bead_handsolder-1206")
+      (reference "L5") (unit 1) (value "Ferrite_Bead_Small") (footprint "Library:ferrite_bead_1206")
     )
     (path "/00000000-0000-0000-0000-000060212678"
@@
       (reference "R57") (unit 1) (value "120r") (footprint "Library:R_0603_1608Metric_fabdesignatorsmall")
     )
-    (path "/00000000-0000-0000-0000-0000617ac9cf"
-      (reference "RS4851") (unit 1) (value "~") (footprint "")
-    )
     (path "/00000000-0000-0000-0000-00005dc0f2c7"

Commit message: arduino version
Parts:
- removed C16: 1u, Library:C_0603_1608Metric_fabdesignatorsmall, symbol PAINTREv3-rescue:C_Small-_saved_synth-cache-instrumnet-rescue
- removed C3, C4, C5: ~, Library:C_0603_1608Metric_fabdesignatorsmall, symbol Device:C
- removed C35: 10n, Library:C_0603_1608Metric_fabdesignatorsmall, symbol PAINTREv3-rescue:C_Small-_saved_synth-cache-instrumnet-rescue
- removed C6: 10u, Library:C_1206_HandSoldering_silkscreenlabel, symbol PAINTREv3-rescue:CP-2164VCA-rescue-instrumnet-rescue
- removed J5: ~, Library:Tag-Connect_TC2030-IDC-NL_2x03_P1.27mm_Vertical, symbol Connector:AVR-ISP-6
- removed L1: ~, Library:ferrite_bead_1206, symbol Device:L
- removed U1: LP2985-5.0, Package_TO_SOT_SMD:SOT-23-5, symbol Regulator_Linear:LP2985-5.0
- removed U2: ~, Package_QFP:TQFP-48_7x7mm_P0.5mm, symbol MCU_Microchip_ATmega:ATmega4809-A
- added A1: Arduino_Nano_Every, Module:Arduino_Nano, symbol MCU_Module:Arduino_Nano_Every
Connections:
- net +5V: now also A1.27 (+5V)
- net GND: now also A1.29 (GND), A1.4 (GND)
- net RS485_EN: now also A1.7 (D4)
- net UART_RX: now also A1.2 (RX1)
- net UART_TX: now also A1.1 (TX1)
- net cipo: now also A1.15 (MISO)
- net copi: now also A1.14 (MOSI)
- net cs_1: now also A1.10 (D7)
- net cs_2: now also A1.11 (D8)
- net cs_3: now also A1.12 (D9)
- net cs_4: now also A1.13 (D10)
- net sck: now also A1.16 (SCK)
- net scl: now also A1.24 (SCL/A5)
- net sda: now also A1.23 (SDA/A4)
- net Vin: now reaches L5.1
- net Vin: now also A1.30 (VIN)
- no-connect marks 1 -> 0
Other:
- note removed: "150mA max draw"
- note removed: "<10mA 328p <10mA BNO080"
- note removed: "ATMEGA4809"
- note removed: "UPDI programming interface (for use with pogo pins, custom setup)"
- note removed: "X7Rs on output, minimum 2.2uF, no maximum bypass C0G"
- note removed: "decoupling pins: 14/15 28/29 42/43"
- moved on the sheet: C7

Commit message: V4 PCB redesign (max ICs)
Parts:
- removed C10, C12, C21, C24, C33: 1u, Library:C_0603_1608Metric_fabdesignatorsmall, symbol Device:C_Small
- removed C11, C13, C14, C15, C23, C30, C31, C32: .1u, Library:C_0603_1608Metric_fabdesignatorsmall, symbol Device:C_Small
- removed J3: TC, Connector_PinHeader_2.54mm:PinHeader_1x16_P2.54mm_Vertical, symbol Connector:Conn_01x16_Male
- removed R10, R11, R19, R21, R26, R36, R37, R38, R39, R48, R49, R50, R51, R9: 50, Library:R_0603_1608Metric_fabdesignatorsmall, symbol PAINTREv3-rescue:R-2164VCA-rescue-instrumnet-rescue
- removed R12, R22, R25, R27, R28, R29, R30, R31, R40, R41, R42, R43, R52: 1M, Library:R_0603_1608Metric_fabdesignatorsmall, symbol PAINTREv3-rescue:R-2164VCA-rescue-instrumnet-rescue
- removed R32, R33, R34, R35, R44, R45, R46, R47, R7, R8: 500, Library:R_0603_1608Metric_fabdesignatorsmall, symbol PAINTREv3-rescue:R-2164VCA-rescue-instrumnet-rescue
- removed U3, U4, U5, U7: ADS1118IDGS, Package_SO:TSSOP-10_3x3mm_P0.5mm, symbol Analog_ADC:ADS1118IDGS
- added C16, C3, C4, C5, C6: .1u, Library:C_0603_1608Metric_fabdesignatorsmall, symbol Device:C_Small
- added J2: TC1, Connector_PinSocket_2.54mm:PinSocket_1x02_P2.54mm_Vertical, symbol Connector:Conn_01x02_Male
- added J3: TC2, Connector_PinSocket_2.54mm:PinSocket_1x02_P2.54mm_Vertical, symbol Connector:Conn_01x02_Male
- added J4: TC3, Connector_PinSocket_2.54mm:PinSocket_1x02_P2.54mm_Vertical, symbol Connector:Conn_01x02_Male
- added J5: TC4, Connector_PinSocket_2.54mm:PinSocket_1x02_P2.54mm_Vertical, symbol Connector:Conn_01x02_Male
- added J6: TC5, Connector_PinSocket_2.54mm:PinSocket_1x02_P2.54mm_Vertical, symbol Connector:Conn_01x02_Male
- added U1, U2, U3, U4, U5: MAX31855KASA, Package_SO:SOIC-8_3.9x4.9mm_P1.27mm, symbol Sensor_Temperature:MAX31855KASA
- C25: value 1u -> .01u
- C26, C27, C28, C29: value .1u -> .01u
- C8, C9: value 1u -> .1u
- R1, R2, R3, R4: value 1M -> 500
- R17, R18: value 50 -> 1M
- U6: footprint Package_SO:SOIC-8_3.9x4.9mm_P1.27mm -> Library:SOT-5X3-8
Connections:
- net tc7+ is gone; now on net +5V: R14.2
- net +5V: now also C17.1, C18.1, C19.1, R16.2, R17.2, R18.2, C16.1, U1.4 (VCC), U2.4 (VCC), U3.4 (VCC), U4.4 (VCC), U5.4 (VCC); no longer R1.1, R14.1, R3.1
- net GND: now also C18.2, C8.1, C9.2, C16.2, C3.1, C4.2, C5.1, C6.2, U1.1 (GND), U2.1 (GND), U3.1 (GND), U4.1 (GND), U5.1 (GND); no longer C18.1, C26.1, C27.2, C28.1, C29.2, R16.2, R2.2, R4.2
- net cipo: now also U1.7 (SO), U2.7 (SO), U3.7 (SO), U4.7 (SO), U5.7 (SO)
- net copi: no longer R18.2
- net cs_1: now also A1.9 (D6), U1.6 (~{CS}); no longer A1.10 (D7)
- net cs_2: now also A1.10 (D7), R14.1, U2.6 (~{CS}); no longer A1.11 (D8)
- net cs_3: now also A1.11 (D8), R16.1, U3.6 (~{CS}); no longer A1.12 (D9)
- net cs_4: now also A1.12 (D9), R17.1, U4.6 (~{CS}); no longer A1.13 (D10)
- net sck: now also U1.5 (SCK), U2.5 (SCK), U3.5 (SCK), U4.5 (SCK), U5.5 (SCK); no longer R17.2
- net tc1+: now also J2.2 (Pin_2)
- net tc1-: now also J2.1 (Pin_1)
- net tc2+: now also J3.1 (Pin_1)
- net tc2-: now also J3.2 (Pin_2); no longer R16.1
- net tc3+: now also R1.1, J4.1 (Pin_1); no longer R1.2, R5.1
- net tc3-: now also J4.2 (Pin_2); no longer R6.1
- net tc4+: now also R3.1, J5.1 (Pin_1); no longer R3.2
- net tc4-: now also J5.2 (Pin_2)
- net tc5+: now also R5.1, J6.1 (Pin_1)
- net tc5-: now also R6.1, J6.2 (Pin_2)
- net cs_5: now reaches R18.1
- net cs_5: now also A1.13 (D10), U5.6 (~{CS})
- net at C20.2, R23.2: now also C25.1, U1.3 (T+)
- net at C22.1, R24.2: now also C25.2, U1.2 (T-)
- net at C2.2, R13.2: now also C27.1, U2.3 (T+)
- net at C34.1, R15.2: now also C27.2, U2.2 (T-)
- net at R5.2: now also C29.1, C8.2, U5.3 (T+); no longer C8.1
- net at C28.2: now also R4.2, C6.1, U4.2 (T-); no longer C25.1
- net at C26.2: now also R2.2, C4.1, U3.2 (T-)
- net at C9.1: now also C29.2, R6.2, U5.2 (T-)
- new net: C26.1, C3.2, R1.2, U3.3 (T+)
- new net: C28.1, C5.2, R3.2, U4.3 (T+)
Other:
- note added: "THVD1400"
- note removed: "THVD1420"
- note removed: "short circuit protection 50 ohms"
- moved on the sheet: C1, R20

Commit message: v4 pcb updates
Parts:
- C36: value ~ -> .1u
Other:
- note added: "7-18V input"
- note removed: "3.6V - 16V input"
- moved on the sheet: H1, H2, H3
Changed lines of the file:
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@@
     (effects (font (size 1.27 1.27)) (justify left bottom))
   )
-  (text "3.6V - 16V input" (at -39.37 31.75 0)
+  (text "7-18V input" (at -19.05 26.67 0)
     (effects (font (size 2.9972 2.9972)) (justify left bottom))
   )
@@
   )
   (text "PAINTREv3 internal instrumentation for HOTROD ice drilling system"
-    (at -177.038 -122.174 0)
+    (at 180.34 387.35 0)
     (effects (font (size 2 2)) (justify left bottom))
   )
@@
       (effects (font (size 1.27 1.27)) (justify left))
     )
-    (property "Value" "~" (id 1) (at 214.249 40.767 0)
+    (property "Value" ".1u" (id 1) (at 214.249 40.767 0)
       (effects (font (size 1.27 1.27)) (justify left))
     )
@@
     (pin "2")
   )
-  (symbol (lib_id "Mechanical:MountingHole") (at -222.25 -107.95 0) (unit 1)
-    (in_bom yes) (on_board yes)
-    (property "Reference" "H3" (id 0) (at -219.71 -109.1184 0)
-      (effects (font (size 1.27 1.27)) (justify left))
-    )
-    (property "Value" "MountingHole" (id 1) (at -219.71 -106.807 0)
-      (effects (font (size 1.27 1.27)) (justify left))
-    )
-    (property "Footprint" "Library:MountingHole_3.2mm_M3" (id 2) (at -222.25 -107.95 0)
-      (effects (font (size 1.27 1.27)) hide)
-    )
-    (property "Datasheet" "~" (id 3) (at -222.25 -107.95 0)
-      (effects (font (size 1.27 1.27)) hide)
-    )
-  )
-  (symbol (lib_id "Mechanical:MountingHole") (at -204.47 -107.95 0) (unit 1)
-    (in_bom yes) (on_board yes)
-    (property "Reference" "H2" (id 0) (at -201.93 -109.1184 0)
-      (effects (font (size 1.27 1.27)) (justify left))
-    )
-    (property "Value" "MountingHole" (id 1) (at -201.93 -106.807 0)
-      (effects (font (size 1.27 1.27)) (justify left))
-    )
-    (property "Footprint" "Library:MountingHole_3.2mm_M3" (id 2) (at -204.47 -107.95 0)
-      (effects (font (size 1.27 1.27)) hide)
-    )
-    (property "Datasheet" "~" (id 3) (at -204.47 -107.95 0)
+  (symbol (lib_id "Mechanical:MountingHole") (at 243.84 359.41 0) (unit 1)
+    (in_bom yes) (on_board yes)
+    (property "Reference" "H3" (id 0) (at 246.38 358.2416 0)
+      (effects (font (size 1.27 1.27)) (justify left))
+    )
+    (property "Value" "MountingHole" (id 1) (at 246.38 360.553 0)
+      (effects (font (size 1.27 1.27)) (justify left))
+    )
+    (property "Footprint" "Library:MountingHole_3.2mm_M3" (id 2) (at 243.84 359.41 0)
+      (effects (font (size 1.27 1.27)) hide)
+    )
+    (property "Datasheet" "~" (id 3) (at 243.84 359.41 0)
+      (effects (font (size 1.27 1.27)) hide)
+    )
+  )
+  (symbol (lib_id "Mechanical:MountingHole") (at 261.62 359.41 0) (unit 1)
+    (in_bom yes) (on_board yes)
+    (property "Reference" "H2" (id 0) (at 264.16 358.2416 0)
+      (effects (font (size 1.27 1.27)) (justify left))
+    )
+    (property "Value" "MountingHole" (id 1) (at 264.16 360.553 0)
+      (effects (font (size 1.27 1.27)) (justify left))
+    )
+    (property "Footprint" "Library:MountingHole_3.2mm_M3" (id 2) (at 261.62 359.41 0)
+      (effects (font (size 1.27 1.27)) hide)
+    )
+    (property "Datasheet" "~" (id 3) (at 261.62 359.41 0)
       (effects (font (size 1.27 1.27)) hide)
     )
@@
     (pin "8")
   )
-  (symbol (lib_id "Mechanical:MountingHole") (at 231.14 17.78 0) (unit 1)
-    (in_bom yes) (on_board yes)
-    (property "Reference" "H1" (id 0) (at 233.68 16.6116 0)
-      (effects (font (size 1.27 1.27)) (justify left))
-    )
-    (property "Value" "~" (id 1) (at 233.68 18.923 0)
-      (effects (font (size 1.27 1.27)) (justify left))
-    )
-    (property "Footprint" "Library:MountingHole_3.2mm_M3" (id 2) (at 231.14 17.78 0)
-      (effects (font (size 1.27 1.27)) hide)
-    )
-    (property "Datasheet" "~" (id 3) (at 231.14 17.78 0)
+  (symbol (lib_id "Mechanical:MountingHole") (at 226.06 359.41 0) (unit 1)
+    (in_bom yes) (on_board yes)
+    (property "Reference" "H1" (id 0) (at 228.6 358.2416 0)
+      (effects (font (size 1.27 1.27)) (justify left))
+    )
+    (property "Value" "~" (id 1) (at 228.6 360.553 0)
+      (effects (font (size 1.27 1.27)) (justify left))
+    )
+    (property "Footprint" "Library:MountingHole_3.2mm_M3" (id 2) (at 226.06 359.41 0)
+      (effects (font (size 1.27 1.27)) hide)
+    )
+    (property "Datasheet" "~" (id 3) (at 226.06 359.41 0)
       (effects (font (size 1.27 1.27)) hide)
     )
@@
     )
     (path "/00000000-0000-0000-0000-00005f729604"
-      (reference "C36") (unit 1) (value "~") (footprint "Library:C_0603_1608Metric_fabdesignatorsmall")
+      (reference "C36") (unit 1) (value ".1u") (footprint "Library:C_0603_1608Metric_fabdesignatorsmall")
     )
     (path "/00000000-0000-0000-0000-00005dc455cc"

Commit message: pv4
Parts:
- removed H2: MountingHole, Library:MountingHole_3.2mm_M3, symbol Mechanical:MountingHole
- added H2: logo, Library:paintre v4 logo, symbol Mechanical:MountingHole_Pad
- R57: footprint Library:R_0603_1608Metric_fabdesignatorsmall -> Resistor_SMD:R_1210_3225Metric_Pad1.30x2.65mm_HandSolder
Other:
- note added: "ADD TERMINATION R AT DATA UNIT ALSO"
Changed lines of the file:
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@@
     (effects (font (size 1.27 1.27)) (justify left bottom))
+  )
+  (text "ADD TERMINATION R AT DATA UNIT ALSO" (at 198.12 21.59 0)
+    (effects (font (size 5 5)) (justify left bottom))
   )
   (text "7-18V input" (at -19.05 26.67 0)
@@
     )
     (property "Datasheet" "~" (id 3) (at 243.84 359.41 0)
-      (effects (font (size 1.27 1.27)) hide)
-    )
-  )
-  (symbol (lib_id "Mechanical:MountingHole") (at 261.62 359.41 0) (unit 1)
-    (in_bom yes) (on_board yes)
-    (property "Reference" "H2" (id 0) (at 264.16 358.2416 0)
-      (effects (font (size 1.27 1.27)) (justify left))
-    )
-    (property "Value" "MountingHole" (id 1) (at 264.16 360.553 0)
-      (effects (font (size 1.27 1.27)) (justify left))
-    )
-    (property "Footprint" "Library:MountingHole_3.2mm_M3" (id 2) (at 261.62 359.41 0)
-      (effects (font (size 1.27 1.27)) hide)
-    )
-    (property "Datasheet" "~" (id 3) (at 261.62 359.41 0)
       (effects (font (size 1.27 1.27)) hide)
     )
@@
       (effects (font (size 1.27 1.27)) (justify left))
     )
-    (property "Footprint" "Library:R_0603_1608Metric_fabdesignatorsmall" (id 2) (at 256.032 30.48 90)
+    (property "Footprint" "Resistor_SMD:R_1210_3225Metric_Pad1.30x2.65mm_HandSolder" (id 2) (at 256.032 30.48 90)
       (effects (font (size 1.27 1.27)) hide)
     )
@@
     (pin "1")
     (pin "2")
+  )
+  (symbol (lib_id "Mechanical:MountingHole_Pad") (at 276.86 363.22 0) (unit 1)
+    (in_bom yes) (on_board yes) (fields_autoplaced)
+    (property "Reference" "H2" (id 0) (at 279.4 360.6799 0)
+      (effects (font (size 1.27 1.27)) (justify left))
+    )
+    (property "Value" "logo" (id 1) (at 279.4 363.2199 0)
+      (effects (font (size 1.27 1.27)) (justify left))
+    )
+    (property "Footprint" "Library:paintre v4 logo" (id 2) (at 276.86 363.22 0)
+      (effects (font (size 1.27 1.27)) hide)
+    )
+    (property "Datasheet" "~" (id 3) (at 276.86 363.22 0)
+      (effects (font (size 1.27 1.27)) hide)
+    )
+    (pin "1")
   )
   (symbol (lib_id "MCU_Module:Arduino_Nano_Every") (at 199.39 217.17 0) (unit 1)
@@
       (reference "H1") (unit 1) (value "~") (footprint "Library:MountingHole_3.2mm_M3")
     )
-    (path "/00000000-0000-0000-0000-00006002e052"
-      (reference "H2") (unit 1) (value "MountingHole") (footprint "Library:MountingHole_3.2mm_M3")
+    (path "/89ea9806-41be-4470-a2cc-12134e415188"
+      (reference "H2") (unit 1) (value "logo") (footprint "Library:paintre v4 logo")
     )
     (path "/00000000-0000-0000-0000-00006002dcf5"
@@
     )
     (path "/00000000-0000-0000-0000-000061901231"
-      (reference "R57") (unit 1) (value "120r") (footprint "Library:R_0603_1608Metric_fabdesignatorsmall")
+      (reference "R57") (unit 1) (value "120r") (footprint "Resistor_SMD:R_1210_3225Metric_Pad1.30x2.65mm_HandSolder")
     )
     (path "/00000000-0000-0000-0000-00005dc0f2c7"
